Commit message: update xacro for experiments. now urdf is dynamically compiled

File: mmseq_assets/thing/xacro/end_effector_fingers.urdf.xacro (robot description, xacro)
@@ -1,9 +1,9 @@
 <?xml version="1.0" encoding="utf-8"?>
 <robot name="end_effector_fingers">
-  <joint name="tool0_tcp_fixed_joint" type="fixed">
-    <origin rpy="0.0 0.0 3.14159" xyz="0.0 0.0 0.290"/>
-    <parent link="ur10_arm_tool0"/>
-    <child link="thing_tool"/>
-  </joint>
+<!--  <joint name="tool0_tcp_fixed_joint" type="fixed">-->
+<!--    <origin rpy="0.0 0.0 3.14159" xyz="0.0 0.0 0.290"/>-->
+<!--    <parent link="ur10_arm_tool0"/>-->
+<!--    <child link="thing_tool"/>-->
+<!--  </joint>-->
   <!-- s = 0.3 -->
   <!-- h = 0.08660254037844387 -->
@@ -15,5 +15,5 @@
   <!-- When oriented forward, the frame has: z forward, x down, y left -->
   <!-- When oriented up (i.e. for balancing): z up, x forward, y left -->
-  <link name="thing_tool">
+  <link name="gripped_object">
     <visual>
       <origin rpy="0 0 0" xyz="0.1155 0 0"/>

Commit message: add rviz visualization. remove old xacro files. rearranged launch files

File: mmseq_assets/thing/xacro/end_effector_fingers.urdf.xacro (robot description, xacro)
@@ -1,4 +1,4 @@
 <?xml version="1.0" encoding="utf-8"?>
-<robot name="end_effector_fingers">
+<robot name="end_effector_fingers" xmlns:xacro="http://wiki.ros.org/xacro">
 <!--  <joint name="tool0_tcp_fixed_joint" type="fixed">-->
 <!--    <origin rpy="0.0 0.0 3.14159" xyz="0.0 0.0 0.290"/>-->
@@ -12,4 +12,9 @@
   <!-- h = 0.0577 -->
   <!-- r = 0.1155 -->
+   <joint name="gripped_object_joint" type="fixed">
+     <xacro:transformed_origin name="gripped_object_transform" />
+     <parent link="gripper"/>
+     <child link="gripped_object"/>
+   </joint>
   <!-- Custom tool for tray balancing -->
   <!-- When oriented forward, the frame has: z forward, x down, y left -->
