Commit message: added box to urdf

File: mmseq_assets/thing/xacro/collision.urdf.xacro (robot description, xacro)
@@ -88,7 +88,7 @@
   </joint>
   <!-- Gripped Object -->
-  <xacro:collision_link_sphere name="gripped_object_collision_link" radius="0.2"/>
+  <xacro:collision_link_sphere name="gripped_object_collision_link" radius="0.22"/>
   <joint name="gripped_object_collision_joint" type="fixed">
-    <origin rpy="0 0 0" xyz="0 0 0.02"/>
+    <origin rpy="0 0 0" xyz="0 0 0.0"/>
     <parent link="gripped_object"/>
     <child link="gripped_object_collision_link"/>

Commit message: replace rack collision cylinder with two spheres.

File: mmseq_assets/thing/xacro/collision.urdf.xacro (robot description, xacro)
@@ -54,4 +54,16 @@
     <parent link="base_link"/>
     <child link="rack_collision_link"/>
+  </joint>
+  <xacro:collision_link_sphere name="rack_collision_link_sphere_1" radius="0.5"/>
+  <joint name="rack_collision_joint_1" type="fixed">
+    <origin rpy="0 0 0" xyz="-0.45 -0.15 0.75"/>
+    <parent link="base_link"/>
+    <child link="rack_collision_link_sphere_1"/>
+  </joint>
+  <xacro:collision_link_sphere name="rack_collision_link_sphere_2" radius="0.5"/>
+  <joint name="rack_collision_joint_2" type="fixed">
+    <origin rpy="0 0 0" xyz="-0.45 0.15 0.75"/>
+    <parent link="base_link"/>
+    <child link="rack_collision_link_sphere_2"/>
   </joint>
   <!-- Collision sphere for the upper arm -->

Commit message: change base collision sphere to one.

File: mmseq_assets/thing/xacro/collision.urdf.xacro (robot description, xacro)
@@ -43,11 +43,11 @@
   </xacro:macro>
   <!-- Collision sphere for the base -->
-  <!-- <xacro:collision_link_sphere name="base_collision_link" radius="0.45"/>
+  <xacro:collision_link_sphere name="base_collision_link" radius="0.45"/>
   <joint name="base_collision_joint" type="fixed">
     <origin rpy="0 0 0" xyz="0 0 -0.08"/>
     <parent link="base_link"/>
     <child link="base_collision_link"/>
-  </joint> -->
-  <xacro:collision_link_sphere name="base_collision_link_front" radius="0.3"/>
+  </joint>
+  <!-- <xacro:collision_link_sphere name="base_collision_link_front" radius="0.3"/>
   <joint name="base_collision_joint_front" type="fixed">
     <origin rpy="0 0 0" xyz="0.35 0 -0.08"/>
@@ -60,5 +60,5 @@
     <parent link="base_link"/>
     <child link="base_collision_link_back"/>
-  </joint>
+  </joint> -->
   <xacro:collision_link_cylinder name="rack_collision_link" radius="0.325"/>
   <joint name="rack_collision_joint" type="fixed">
