Commit message: added restaurant scene

File: mmseq_assets/scenes/xacro/simple_obstacles.urdf.xacro (robot description, xacro)
@@ -18,21 +18,32 @@
   </xacro:macro>
   <link name="obstacle_base_link"/>
-  <xacro:obstacle_link name="obstacle_link_1" material="red">
+<!--  <xacro:obstacle_link name="obstacle_link_1" material="red">-->
+<!--    <geometry>-->
+<!--      <sphere radius="0.5"/>-->
+<!--    </geometry>-->
+<!--  </xacro:obstacle_link>-->
+<!--  <joint name="obstacle_joint_1" type="fixed">-->
+<!--    <origin rpy="0 0 0" xyz="2 0 0"/>-->
+<!--    <parent link="obstacle_base_link"/>-->
+<!--    <child link="obstacle_link_1"/>-->
+<!--  </joint>-->
+<!--  <xacro:obstacle_link name="obstacle_link_2" material="red">-->
+<!--    <geometry>-->
+<!--      <sphere radius="0.25"/>-->
+<!--    </geometry>-->
+<!--  </xacro:obstacle_link>-->
+<!--  <joint name="obstacle_joint_2" type="fixed">-->
+<!--    <origin rpy="0 0 0" xyz="1 1 1"/>-->
+<!--    <parent link="obstacle_base_link"/>-->
+<!--    <child link="obstacle_link_2"/>-->
+<!--  </joint>-->
+    <xacro:obstacle_link name="obstacle_link_2" material="red">
     <geometry>
-      <sphere radius="0.5"/>
-    </geometry>
-  </xacro:obstacle_link>
-  <joint name="obstacle_joint_1" type="fixed">
-    <origin rpy="0 0 0" xyz="2 0 0"/>
-    <parent link="obstacle_base_link"/>
-    <child link="obstacle_link_1"/>
-  </joint>
-  <xacro:obstacle_link name="obstacle_link_2" material="red">
-    <geometry>
-      <sphere radius="0.25"/>
+      <cylinder radius="0.25" length="1."/>
+<!--      <sphere radius="0.25"/>-->
     </geometry>
   </xacro:obstacle_link>
   <joint name="obstacle_joint_2" type="fixed">
-    <origin rpy="0 0 0" xyz="1 1 1"/>
+    <origin rpy="0 0 0" xyz="5.0 0.5 0.5"/>
     <parent link="obstacle_base_link"/>
     <child link="obstacle_link_2"/>
@@ -40,10 +51,10 @@
   <xacro:obstacle_link name="obstacle_link_3" material="red">
     <geometry>
-      <cylinder radius="0.5" length="1."/>
+      <cylinder radius="0.25" length="1."/>
 <!--      <sphere radius="0.25"/>-->
     </geometry>
   </xacro:obstacle_link>
   <joint name="obstacle_joint_3" type="fixed">
-    <origin rpy="0 0 0" xyz="0 -2 0.5"/>
+    <origin rpy="0 0 0" xyz="3.0 -0.5 0.5"/>
     <parent link="obstacle_base_link"/>
     <child link="obstacle_link_3"/>
